Commit message: working real robot

File: description/robot_core.xacro (robot description, xacro)
@@ -21,5 +21,5 @@
         <parent link="base_link" />
         <child link="chassis" />
-        <origin xyz="-0.065 0 0"/>
+        <origin xyz="-0.1375 0 0"/>
     </joint>
     <link name="chassis">
@@ -55,5 +55,5 @@
             <origin xyz="0 0 0"/>
             <geometry>
-                <cylinder radius="0.0325" length="0.025"/>
+                <cylinder radius="0.032" length="0.025"/>
             </geometry>
             <material name="blue"/>
@@ -62,8 +62,8 @@
             <origin xyz="0 0 0"/>
             <geometry>
-                <sphere radius="0.0325"/>
+                <sphere radius="0.032"/>
             </geometry>
         </collision>
-        <xacro:inertial_cylinder mass="0.1" radius="0.0325" length="0.025">
+        <xacro:inertial_cylinder mass="0.1" radius="0.032" length="0.025">
             <origin xyz="0 0 0" rpy="0 0 0"/>
         </xacro:inertial_cylinder>
@@ -83,5 +83,5 @@
             <origin xyz="0 0 0"/>
             <geometry>
-                <cylinder radius="0.0325" length="0.025"/>
+                <cylinder radius="0.032" length="0.025"/>
             </geometry>
             <material name="blue"/>
@@ -90,8 +90,8 @@
             <origin xyz="0 0 0"/>
             <geometry>
-                <sphere radius="0.0325"/>
+                <sphere radius="0.032"/>
             </geometry>
         </collision>
-        <xacro:inertial_cylinder mass="0.1" radius="0.0325" length="0.025">
+        <xacro:inertial_cylinder mass="0.1" radius="0.032" length="0.025">
             <origin xyz="0 0 0" rpy="0 0 0"/>
         </xacro:inertial_cylinder>
@@ -104,5 +104,5 @@
         <parent link="chassis"/>
         <child link="caster_wheel"/>
-        <origin xyz="0.155 0 0"/>
+        <origin xyz="0.045 0 0"/>
     </joint>
     <link name="caster_wheel">

File: description/ros2_control.xacro (robot description, xacro)
@@ -1,5 +1,33 @@
 <?xml version="1.0"?>
 <robot xmlns:xacro="http://www.ros.org/wiki/xacro">
-    <ros2_control name="GazeboSystem" type="system">
+    <ros2_control name="RealRobot" type="system">
+        <hardware>
+            <plugin>diffdrive_esp/DiffDriveEspHardware</plugin>
+            <param name="left_wheel_name">left_wheel_joint</param>
+            <param name="right_wheel_name">right_wheel_joint</param>
+            <param name="loop_rate">30</param>
+            <param name="device">/dev/ttyAMA0</param>
+            <param name="baud_rate">115200</param>
+            <param name="timeout_ms">1000</param>
+            <param name="enc_counts_per_rev">2184</param>
+        </hardware>
+        <joint name="left_wheel_joint">
+            <command_interface name="velocity">
+                <param name="min">-10</param>
+                <param name="max">10</param>
+            </command_interface>
+            <state_interface name="position"/>
+            <state_interface name="velocity"/>
+        </joint>
+        <joint name="right_wheel_joint">
+            <command_interface name="velocity">
+                <param name="min">-10</param>
+                <param name="max">10</param>
+            </command_interface>
+            <state_interface name="position" />
+            <state_interface name="velocity" />
+        </joint>
+    </ros2_control>
+    <!-- <ros2_control name="GazeboSystem" type="system">
         <hardware>
             <plugin>gazebo_ros2_control/GazeboSystem</plugin>
@@ -21,5 +49,5 @@
             <state_interface name="velocity" />
         </joint>
-    </ros2_control>
+    </ros2_control> -->
     <gazebo>
         <plugin name="gazebo_ros2_control" filename="libgazebo_ros2_control.so">
