Commit message: Added camera, changed robot color.

File: description/robot.urdf.xacro (robot description, xacro)
@@ -4,4 +4,5 @@
     <xacro:arg name="sim_mode" default="false"/>
     <xacro:include filename="robot_core.xacro" />
+    <xacro:include filename="camera.xacro" />
     <xacro:if value="$(arg use_ros2_control)">
         <xacro:include filename="ros2_control.xacro" />

File: description/robot_core.xacro (robot description, xacro)
@@ -13,4 +13,7 @@
     <material name="blue">
         <color rgba="0 0 1 1" />
+    </material>
+    <material name="red">
+        <color rgba="1 0 0 1" />
     </material>
     <!-- BASE LINK -->
@@ -42,5 +45,5 @@
     </link>
     <gazebo reference="chassis">
-        <material>Gazebo/Gray</material>
+        <material>Gazebo/DarkGrey</material>
     </gazebo>
     <!-- LEFT WHEEL LINK -->

File: description/ros2_control.xacro (robot description, xacro)
@@ -1,5 +1,5 @@
 <?xml version="1.0"?>
 <robot xmlns:xacro="http://www.ros.org/wiki/xacro">
-    <ros2_control name="RealRobot" type="system">
+    <!-- <ros2_control name="RealRobot" type="system">
         <hardware>
             <plugin>diffdrive_esp/DiffDriveEspHardware</plugin>
@@ -28,6 +28,6 @@
             <state_interface name="velocity" />
         </joint>
-    </ros2_control>
-    <!-- <ros2_control name="GazeboSystem" type="system">
+    </ros2_control> -->
+    <ros2_control name="GazeboSystem" type="system">
         <hardware>
             <plugin>gazebo_ros2_control/GazeboSystem</plugin>
@@ -49,5 +49,5 @@
             <state_interface name="velocity" />
         </joint>
-    </ros2_control> -->
+    </ros2_control>
     <gazebo>
         <plugin name="gazebo_ros2_control" filename="libgazebo_ros2_control.so">
